Commit message: combine new find_bloc_noDepth file and new launch file

File: src/sagittarius_descriptions/urdf/sgr532.urdf.xacro (robot description, xacro)
@@ -650,5 +650,5 @@
   <link name="$(arg robot_name)/usb_cam_link"></link>
   <joint name="joint_usb_cam_frame" type="fixed">
-    <origin xyz="0.05 0 0.05825" rpy="-1.57 0 -1.57" />
+    <origin xyz="0.05 0.032 0.1" rpy="-1.57 0 -1.57" />
     <parent link="$(arg robot_name)/link6" />
     <child link="$(arg robot_name)/usb_cam_link" />
