Commit message: Updated camera position in urdf TF tree

File: src/sagittarius_pcks/sagittarius_descriptions/urdf/sgr532.urdf.xacro (robot description, xacro)
@@ -650,5 +650,5 @@
   <link name="$(arg robot_name)/usb_cam_link"></link>
   <joint name="joint_usb_cam_frame" type="fixed">
-    <origin xyz="0.05 0 0.05825" rpy="-1.57 0 -1.57" />
+    <origin xyz="0.05 0 0.1" rpy="-1.57 0 -1.57" />
     <parent link="$(arg robot_name)/link6" />
     <child link="$(arg robot_name)/usb_cam_link" />

Commit message: Updated y position of camera

File: src/sagittarius_pcks/sagittarius_descriptions/urdf/sgr532.urdf.xacro (robot description, xacro)
@@ -650,5 +650,5 @@
   <link name="$(arg robot_name)/usb_cam_link"></link>
   <joint name="joint_usb_cam_frame" type="fixed">
-    <origin xyz="0.05 0 0.1" rpy="-1.57 0 -1.57" />
+    <origin xyz="0.05 0.032 0.1" rpy="-1.57 0 -1.57" />
     <parent link="$(arg robot_name)/link6" />
     <child link="$(arg robot_name)/usb_cam_link" />

Commit message: successfully stack four bricks 0222

File: src/sagittarius_pcks/sagittarius_descriptions/urdf/sgr532.urdf.xacro (robot description, xacro)
@@ -650,5 +650,5 @@
   <link name="$(arg robot_name)/usb_cam_link"></link>
   <joint name="joint_usb_cam_frame" type="fixed">
-    <origin xyz="0.05 0.032 0.1" rpy="-1.57 0 -1.57" />
+    <origin xyz="0.065 0.032 0.097" rpy="-1.543 -0.056 -1.489" />
     <parent link="$(arg robot_name)/link6" />
     <child link="$(arg robot_name)/usb_cam_link" />

Commit message: add rotation

File: src/sagittarius_pcks/sagittarius_descriptions/urdf/sgr532.urdf.xacro (robot description, xacro)
@@ -500,5 +500,5 @@
     type="fixed">
     <origin
-      xyz="0.0557 0 0"
+      xyz="0.1137 0 0"
       rpy="0 0 0" />
     <parent
@@ -650,5 +650,5 @@
   <link name="$(arg robot_name)/usb_cam_link"></link>
   <joint name="joint_usb_cam_frame" type="fixed">
-    <origin xyz="0.065 0.032 0.097" rpy="-1.543 -0.056 -1.489" />
+    <origin xyz="0.065 0.033 0.101" rpy="-1.567 -0.057 -1.496" />
     <parent link="$(arg robot_name)/link6" />
     <child link="$(arg robot_name)/usb_cam_link" />
@@ -656,4 +656,12 @@
     <limit lower="0" upper="0" effort="0" velocity="0" />
   </joint>
+  <!-- <link name="$(arg robot_name)/end_effector"></link>
+  <joint name="joint_end_effector" type="fixed">
+    <origin xyz="0.1137 0 0" rpy="0 0 0" />
+    <parent link="$(arg robot_name)/link6" />
+    <child link="$(arg robot_name)/end_effector" />
+    <axis xyz="0 0 0" />
+    <limit lower="0" upper="0" effort="0" velocity="0" />
+  </joint> -->
   <xacro:if value="${urdf_loc != ''}">
     <xacro:include filename="${urdf_loc}"/>

Commit message: rotate two times before pick up

File: src/sagittarius_pcks/sagittarius_descriptions/urdf/sgr532.urdf.xacro (robot description, xacro)
@@ -650,5 +650,5 @@
   <link name="$(arg robot_name)/usb_cam_link"></link>
   <joint name="joint_usb_cam_frame" type="fixed">
-    <origin xyz="0.065 0.033 0.101" rpy="-1.567 -0.057 -1.496" />
+    <origin xyz="0.062 0.026 0.106" rpy="-1.572 -0.047 -1.453" />
     <parent link="$(arg robot_name)/link6" />
     <child link="$(arg robot_name)/usb_cam_link" />

Commit message: Mar1 add lookaroun function and stack great except little jump in drop goal action

File: src/sagittarius_pcks/sagittarius_descriptions/urdf/sgr532.urdf.xacro (robot description, xacro)
@@ -650,5 +650,5 @@
   <link name="$(arg robot_name)/usb_cam_link"></link>
   <joint name="joint_usb_cam_frame" type="fixed">
-    <origin xyz="0.062 0.026 0.106" rpy="-1.572 -0.047 -1.453" />
+    <origin xyz="0.064 0.028 0.102" rpy="-1.534 -0.051 -1.481" />
     <parent link="$(arg robot_name)/link6" />
     <child link="$(arg robot_name)/usb_cam_link" />

Commit message: update urdf end effector position

File: src/sagittarius_pcks/sagittarius_descriptions/urdf/sgr532.urdf.xacro (robot description, xacro)
@@ -500,5 +500,5 @@
     type="fixed">
     <origin
-      xyz="0.0557 0 0"
+      xyz="0.1137 0 0"
       rpy="0 0 0" />
     <parent
@@ -650,5 +650,5 @@
   <link name="$(arg robot_name)/usb_cam_link"></link>
   <joint name="joint_usb_cam_frame" type="fixed">
-    <origin xyz="0.05 0.032 0.1" rpy="-1.57 0 -1.57" />
+    <origin xyz="0.064 0.028 0.102" rpy="-1.534 -0.051 -1.481" />
     <parent link="$(arg robot_name)/link6" />
     <child link="$(arg robot_name)/usb_cam_link" />
@@ -656,4 +656,12 @@
     <limit lower="0" upper="0" effort="0" velocity="0" />
   </joint>
+  <!-- <link name="$(arg robot_name)/end_effector"></link>
+  <joint name="joint_end_effector" type="fixed">
+    <origin xyz="0.1137 0 0" rpy="0 0 0" />
+    <parent link="$(arg robot_name)/link6" />
+    <child link="$(arg robot_name)/end_effector" />
+    <axis xyz="0 0 0" />
+    <limit lower="0" upper="0" effort="0" velocity="0" />
+  </joint> -->
   <xacro:if value="${urdf_loc != ''}">
     <xacro:include filename="${urdf_loc}"/>

Commit message: Integrated everything on main branch, added camera inertia estimate

File: src/sagittarius_pcks/sagittarius_descriptions/urdf/sgr532.urdf.xacro (robot description, xacro)
@@ -648,7 +648,22 @@
     </actuator>
   </transmission>
-  <link name="$(arg robot_name)/usb_cam_link"></link>
+  <link name="$(arg robot_name)/usb_cam_link">
+    <inertial>
+      <origin
+        xyz="0 0 0"
+        rpy="0 0 0" />
+      <mass
+        value="0.561320558" />
+      <inertia
+        ixx="8.42E-5"
+        ixy="0.0"
+        ixz="0.0"
+        iyy="8.42E-5"
+        iyz="0.0"
+        izz="8.42E-5" />
+    </inertial>
+  </link>
   <joint name="joint_usb_cam_frame" type="fixed">
-    <origin xyz="0.064 0.028 0.102" rpy="-1.534 -0.051 -1.481" />
+    <origin xyz="0.069 0.029 0.114" rpy="-1.745 -0.036 -1.491" />
     <parent link="$(arg robot_name)/link6" />
     <child link="$(arg robot_name)/usb_cam_link" />

Commit message: go1 with move_base

File: src/sagittarius_pcks/sagittarius_descriptions/urdf/sgr532.urdf.xacro (robot description, xacro)
@@ -650,5 +650,5 @@
   <link name="$(arg robot_name)/usb_cam_link"></link>
   <joint name="joint_usb_cam_frame" type="fixed">
-    <origin xyz="0.062 0.026 0.106" rpy="-1.572 -0.047 -1.453" />
+    <origin xyz="0.065 0.04 0.104" rpy="-1.513 -0.038 -1.546" />
     <parent link="$(arg robot_name)/link6" />
     <child link="$(arg robot_name)/usb_cam_link" />

Commit message: Working 4-layered colorful wall demo

File: src/sagittarius_pcks/sagittarius_descriptions/urdf/sgr532.urdf.xacro (robot description, xacro)
@@ -665,5 +665,5 @@
   </link>
   <joint name="joint_usb_cam_frame" type="fixed">
-    <origin xyz="0.069 0.029 0.114" rpy="-1.745 -0.036 -1.491" />
+    <origin xyz="0.063 0.033 0.110" rpy="-1.626 -0.028 -1.524" />
     <parent link="$(arg robot_name)/link6" />
     <child link="$(arg robot_name)/usb_cam_link" />

Commit message: change the name of the ros_example_walk to quadruped_PID_walk

File: src/sagittarius_pcks/sagittarius_descriptions/urdf/sgr532.urdf.xacro (robot description, xacro)
@@ -665,5 +665,5 @@
   </link>
   <joint name="joint_usb_cam_frame" type="fixed">
-    <origin xyz="0.063 0.033 0.110" rpy="-1.626 -0.028 -1.524" />
+    <origin xyz="0.062 0.033 0.095" rpy="1.064 -1.516 0.551" />
     <parent link="$(arg robot_name)/link6" />
     <child link="$(arg robot_name)/usb_cam_link" />

Commit message: successfully build a green brick and ask ped to move to the desired point and drop but still need recalibration for exposure

File: src/sagittarius_pcks/sagittarius_descriptions/urdf/sgr532.urdf.xacro (robot description, xacro)
@@ -665,5 +665,6 @@
   </link>
   <joint name="joint_usb_cam_frame" type="fixed">
-    <origin xyz="0.062 0.033 0.095" rpy="1.064 -1.516 0.551" />
+    <!-- <origin xyz="0.048 0.047 0.095" rpy="-1.62 -0.021 -1.517" /> -->
+    <origin xyz="0.063 0.033 0.100" rpy="-1.626 -0.028 -1.524" />
     <parent link="$(arg robot_name)/link6" />
     <child link="$(arg robot_name)/usb_cam_link" />

Commit message: fix the angle of UWB

File: src/sagittarius_pcks/sagittarius_descriptions/urdf/sgr532.urdf.xacro (robot description, xacro)
@@ -665,5 +665,4 @@
   </link>
   <joint name="joint_usb_cam_frame" type="fixed">
-    <!-- <origin xyz="0.048 0.047 0.095" rpy="-1.62 -0.021 -1.517" /> -->
     <origin xyz="0.063 0.033 0.100" rpy="-1.626 -0.028 -1.524" />
     <parent link="$(arg robot_name)/link6" />
